File: hardware/stm32_ds2480_emu.sch (KiCad schematic (older format))
At the start: 26 parts, among them J1 USB_B_Micro, J2 SWD, J3 Pull-Up, J4 OW, Q1 SI2302CDS, SW1 BOOT, U1 AP2204K-3.3, U2 STM32F042F6Px

Commit message: Firmware added
Parts:
- D2: Part Number LTST-C170KRKT -> LTST-C170KGKT
- D3: Part Number LTST-C170KGKT -> LTST-C170KRKT
- R2, R3: Part Number 0603SAF1000T5E -> 0603SAJ0101T5E
- R5, R6: Part Number 0603SAJ047JT5E -> 0805S8J047JT5E
Changed lines of the file:
@@
 F 3 "~" H 9450 4750 50  0001 C CNN
 F 4 "ROYALOHM" H 9450 4750 50  0001 C CNN "Brand"
-F 5 "0603SAJ047JT5E" H 9450 4750 50  0001 C CNN "Part Number"
+F 5 "0805S8J047JT5E" H 9450 4750 50  0001 C CNN "Part Number"
 	1    9450 4750
 	0    1    1    0
@@
 F 3 "~" H 9450 5450 50  0001 C CNN
 F 4 "ROYALOHM" H 9450 5450 50  0001 C CNN "Brand"
-F 5 "0603SAJ047JT5E" H 9450 5450 50  0001 C CNN "Part Number"
+F 5 "0805S8J047JT5E" H 9450 5450 50  0001 C CNN "Part Number"
 	1    9450 5450
 	0    1    1    0
@@
 F 3 "~" H 5200 6400 50  0001 C CNN
 F 4 "ROYALOHM" H 5200 6400 50  0001 C CNN "Brand"
-F 5 "0603SAF1000T5E" H 5200 6400 50  0001 C CNN "Part Number"
+F 5 "0603SAJ0101T5E" H 5200 6400 50  0001 C CNN "Part Number"
 	1    5200 6400
 	1    0    0    -1
@@
 F 3 "~" H 5200 5900 50  0001 C CNN
 F 4 "LITEON" H 5200 5900 50  0001 C CNN "Brand"
-F 5 "LTST-C170KRKT" H 5200 5900 50  0001 C CNN "Part Number"
+F 5 "LTST-C170KGKT" H 5200 5900 50  0001 C CNN "Part Number"
 	1    5200 5900
 	0    -1   -1   0
@@
 F 3 "~" H 5750 6400 50  0001 C CNN
 F 4 "ROYALOHM" H 5750 6400 50  0001 C CNN "Brand"
-F 5 "0603SAF1000T5E" H 5750 6400 50  0001 C CNN "Part Number"
+F 5 "0603SAJ0101T5E" H 5750 6400 50  0001 C CNN "Part Number"
 	1    5750 6400
 	1    0    0    -1
@@
 Wire Wire Line
 	6200 1750 5600 1750
+Text Label 5700 1650 0    50   ~ 0
+SYS_SWDIO
 Text Label 5700 1750 0    50   ~ 0
-SYS_SWDIO
-Text Label 5700 1650 0    50   ~ 0
 SYS_SWCLK
 NoConn ~ 5900 3650
@@
 F 3 "~" H 5750 5900 50  0001 C CNN
 F 4 "LITEON" H 5750 5900 50  0001 C CNN "Brand"
-F 5 "LTST-C170KGKT" H 5750 5900 50  0001 C CNN "Part Number"
+F 5 "LTST-C170KRKT" H 5750 5900 50  0001 C CNN "Part Number"
 	1    5750 5900
 	0    -1   -1   0

Commit message: All componenets moved to top side
Parts:
- J4: renamed from J2; footprint Connector_PinHeader_2.54mm:PinHeader_1x04_P2.54mm_Vertical -> Connector_PinHeader_1.27mm:PinHeader_1x05_P1.27mm_Vertical; symbol Connector_Generic:Conn_01x04 -> Connector_Generic:Conn_01x05; Brand KLS ELECTRONIC -> (none); Part Number L-KLS1-207-1-04-S -> (none)
- TP1: renamed from TP2; value OW-SYNC -> SYNC
- renumbered D2 to D1, D3 to D2, D4 to D3, D1 to D4, J3 to J1, J4 to J2, J1 to J3, R7 to R1, R5 to R4, R4 to R5, R1 to R7, TP1 to TP2
Connections:
- net labels added: NRST
- wire segments 98 -> 99
Other:
- moved on the sheet: F1, TP2
Changed lines of the file:
@@
 EESchema Schematic File Version 4
 LIBS:stm32_ds2480_emu-cache
-EELAYER 29 0
+EELAYER 30 0
 EELAYER END
 $Descr A4 11693 8268
@@
 $EndDescr
 $Comp
-L Device:R R5
+L Device:R R4
 U 1 1 5CAFA495
 P 9450 4750
-F 0 "R5" V 9243 4750 50  0000 C CNN
+F 0 "R4" V 9243 4750 50  0000 C CNN
 F 1 "4.7R" V 9334 4750 50  0000 C CNN
 F 2 "Resistor_SMD:R_0805_2012Metric" V 9380 4750 50  0001 C CNN
@@
 	9100 5450 9100 5650
 $Comp
-L Power_Protection:SP0503BAHT D1
+L Power_Protection:SP0503BAHT D4
 U 1 1 5CB5E302
 P 2700 6050
-F 0 "D1" H 2905 6096 50  0000 L CNN
+F 0 "D4" H 2905 6096 50  0000 L CNN
 F 1 "SP0503BAHT" H 2905 6005 50  0000 L CNN
 F 2 "Package_TO_SOT_SMD:SOT-143" H 2925 6000 50  0001 L CNN
@@
 $EndComp
 $Comp
-L Connector:USB_B_Micro J1
+L Connector:USB_B_Micro J3
 U 1 1 5CB5F1D0
 P 1900 5550
-F 0 "J1" H 1957 6017 50  0000 C CNN
+F 0 "J3" H 1957 6017 50  0000 C CNN
 F 1 "USB_B_Micro" H 1957 5926 50  0000 C CNN
 F 2 "Connector_USB:USB_Micro-B_Molex-105017-0001" H 2050 5500 50  0001 C CNN
@@
 NoConn ~ 2200 5750
 Wire Wire Line
-	2200 5350 2800 5350
-Wire Wire Line
-	2200 5550 2600 5550
-Wire Wire Line
-	2800 5350 2800 5150
+	2200 5350 2600 5350
+Wire Wire Line
+	2600 5350 2600 5150
 Wire Wire Line
 	2700 6250 2700 6450
@@
 L Device:Polyfuse F1
 U 1 1 5CB6BBAF
-P 2800 5000
-F 0 "F1" H 2888 5046 50  0000 L CNN
-F 1 "Polyfuse" H 2888 4955 50  0000 L CNN
-F 2 "Fuse:Fuse_1206_3216Metric" H 2850 4800 50  0001 L CNN
-F 3 "~" H 2800 5000 50  0001 C CNN
-F 4 "BOURNS" H 2800 5000 50  0001 C CNN "Brand"
-F 5 "MF-NSMF012-2" H 2800 5000 50  0001 C CNN "Part Number"
-	1    2800 5000
+P 2600 5000
+F 0 "F1" H 2688 5046 50  0000 L CNN
+F 1 "Polyfuse" H 2688 4955 50  0000 L CNN
+F 2 "Fuse:Fuse_1206_3216Metric" H 2650 4800 50  0001 L CNN
+F 3 "~" H 2600 5000 50  0001 C CNN
+F 4 "BOURNS" H 2600 5000 50  0001 C CNN "Brand"
+F 5 "MF-NSMF012-2" H 2600 5000 50  0001 C CNN "Part Number"
+	1    2600 5000
 	1    0    0    -1
 $EndComp
@@
 USB_N
 Wire Wire Line
-	2800 4850 2800 4650
+	2600 4850 2600 4650
 $Comp
 L power:+5V #PWR05
 U 1 1 5CBC6C1D
-P 2800 4450
-F 0 "#PWR05" H 2800 4300 50  0001 C CNN
-F 1 "+5V" H 2815 4623 50  0000 C CNN
-F 2 "" H 2800 4450 50  0001 C CNN
-F 3 "" H 2800 4450 50  0001 C CNN
-	1    2800 4450
-	1    0    0    -1
-$EndComp
-Wire Wire Line
-	2800 4650 3000 4650
-Connection ~ 2800 4650
-Wire Wire Line
-	2800 4650 2800 4450
+P 2600 4450
+F 0 "#PWR05" H 2600 4300 50  0001 C CNN
+F 1 "+5V" H 2615 4623 50  0000 C CNN
+F 2 "" H 2600 4450 50  0001 C CNN
+F 3 "" H 2600 4450 50  0001 C CNN
+	1    2600 4450
+	1    0    0    -1
+$EndComp
+Wire Wire Line
+	2600 4650 2800 4650
+Connection ~ 2600 4650
+Wire Wire Line
+	2600 4650 2600 4450
 $Comp
 L power:PWR_FLAG #FLG01
 U 1 1 5CBCC599
-P 3000 4650
-F 0 "#FLG01" H 3000 4725 50  0001 C CNN
-F 1 "PWR_FLAG" V 3000 4778 50  0000 L CNN
-F 2 "" H 3000 4650 50  0001 C CNN
-F 3 "~" H 3000 4650 50  0001 C CNN
-	1    3000 4650
+P 2800 4650
+F 0 "#FLG01" H 2800 4725 50  0001 C CNN
+F 1 "PWR_FLAG" V 2800 4778 50  0000 L CNN
+F 2 "" H 2800 4650 50  0001 C CNN
+F 3 "~" H 2800 4650 50  0001 C CNN
+	1    2800 4650
 	0    1    1    0
 $EndComp
 $Comp
-L Device:D_Zener D4
+L Device:D_Zener D3
 U 1 1 5CAD732E
 P 9100 5100
-F 0 "D4" V 9054 5179 50  0000 L CNN
+F 0 "D3" V 9054 5179 50  0000 L CNN
 F 1 "5.1V" V 9145 5179 50  0000 L CNN
 F 2 "Diode_SMD:D_SOT-23_ANK" H 9100 5100 50  0001 C CNN
@@
 	9800 5050 9900 5050
 $Comp
-L Connector_Generic:Conn_01x02 J4
+L Connector_Generic:Conn_01x02 J2
 U 1 1 5CAD1933
 P 10100 5050
-F 0 "J4" H 10180 5042 50  0000 L CNN
+F 0 "J2" H 10180 5042 50  0000 L CNN
 F 1 "OW" H 10180 4951 50  0000 L CNN
 F 2 "Connector_JST:JST_XH_B02B-XH-A_1x02_P2.50mm_Vertical" H 10100 5050 50  0001 C CNN
@@
 NoConn ~ 4700 4150
 $Comp
-L Connector:TestPoint TP1
+L Connector:TestPoint TP2
 U 1 1 5CCC669F
-P 4500 3150
-F 0 "TP1" V 4550 3450 50  0000 C CNN
-F 1 "NRST" V 4450 3450 50  0000 C CNN
-F 2 "TestPoint:TestPoint_Pad_D1.5mm" H 4700 3150 50  0001 C CNN
-F 3 "~" H 4700 3150 50  0001 C CNN
-	1    4500 3150
+P 4300 3150
+F 0 "TP2" V 4350 3450 50  0000 C CNN
+F 1 "NRST" V 4250 3450 50  0000 C CNN
+F 2 "TestPoint:TestPoint_Pad_D1.5mm" H 4500 3150 50  0001 C CNN
+F 3 "~" H 4500 3150 50  0001 C CNN
+	1    4300 3150
 	0    -1   -1   0
 $EndComp
 Wire Wire Line
-	4700 3150 4500 3150
+	4700 3150 4300 3150
 Text Label 6000 4150 0    50   ~ 0
 SYS_SWDIO
@@
 	5200 6050 5200 6250
 $Comp
-L Device:LED D2
+L Device:LED D1
 U 1 1 5CCF8464
 P 5200 5900
-F 0 "D2" V 5239 5783 50  0000 R CNN
+F 0 "D1" V 5239 5783 50  0000 R CNN
 F 1 "LED1" V 5148 5783 50  0000 R CNN
 F 2 "LED_SMD:LED_0805_2012Metric" H 5200 5900 50  0001 C CNN
@@
 $EndComp
 $Comp
-L Device:R R1
+L Device:R R7
 U 1 1 5CB1151A
 P 4700 6700
-F 0 "R1" H 4770 6746 50  0000 L CNN
+F 0 "R7" H 4770 6746 50  0000 L CNN
 F 1 "10K" H 4770 6655 50  0000 L CNN
 F 2 "Resistor_SMD:R_0603_1608Metric" V 4630 6700 50  0001 C CNN
@@
 	9850 2300 9750 2300
 $Comp
-L Connector_Generic:Conn_01x02 J3
+L Connector_Generic:Conn_01x02 J1
 U 1 1 5CAD96D7
 P 10050 2300
-F 0 "J3" H 10130 2342 50  0000 L CNN
+F 0 "J1" H 10130 2342 50  0000 L CNN
 F 1 "Pull-Up" H 10130 2251 50  0000 L CNN
 F 2 "Connector_PinHeader_2.54mm:PinHeader_1x02_P2.54mm_Vertical" H 10050 2300 50  0001 C CNN
@@
 $EndComp
 $Comp
-L Device:R R7
+L Device:R R1
 U 1 1 5CADD3FB
 P 9750 2750
-F 0 "R7" H 9820 2796 50  0000 L CNN
+F 0 "R1" H 9820 2796 50  0000 L CNN
 F 1 "2.2K" H 9820 2705 50  0000 L CNN
 F 2 "Resistor_SMD:R_0805_2012Metric" V 9680 2750 50  0001 C CNN
@@
 	9350 2800 9350 2400
 $Comp
-L Device:R R4
+L Device:R R5
 U 1 1 5CAD4566
 P 8950 2750
-F 0 "R4" H 9020 2796 50  0000 L CNN
+F 0 "R5" H 9020 2796 50  0000 L CNN
 F 1 "10K" H 9020 2705 50  0000 L CNN
 F 2 "Resistor_SMD:R_0603_1608Metric" V 8880 2750 50  0001 C CNN
@@
 $EndComp
 $Comp
-L Connector_Generic:Conn_01x04 J2
+L Connector_Generic:Conn_01x05 J4
 U 1 1 5CCA7536
-P 6400 1650
-F 0 "J2" H 6480 1642 50  0000 L CNN
-F 1 "SWD" H 6480 1551 50  0000 L CNN
-F 2 "Connector_PinHeader_2.54mm:PinHeader_1x04_P2.54mm_Vertical" H 6400 1650 50  0001 C CNN
-F 3 "~" H 6400 1650 50  0001 C CNN
-F 4 "KLS ELECTRONIC" H 6400 1650 50  0001 C CNN "Brand"
-F 5 "L-KLS1-207-1-04-S" H 6400 1650 50  0001 C CNN "Part Number"
-	1    6400 1650
-	1    0    0    -1
-$EndComp
-Wire Wire Line
-	6200 1850 6000 1850
-Wire Wire Line
-	6000 1850 6000 2050
+P 6400 1750
+F 0 "J4" H 6480 1742 50  0000 L CNN
+F 1 "SWD" H 6480 1651 50  0000 L CNN
+F 2 "Connector_PinHeader_1.27mm:PinHeader_1x05_P1.27mm_Vertical" H 6400 1750 50  0001 C CNN
+F 3 "~" H 6400 1750 50  0001 C CNN
+F 4 "" H 6400 1750 50  0001 C CNN "Brand"
+F 5 "" H 6400 1750 50  0001 C CNN "Part Number"
+	1    6400 1750
+	1    0    0    -1
+$EndComp
+Wire Wire Line
+	6200 1950 6000 1950
+Wire Wire Line
+	6000 1950 6000 2150
 $Comp
 L power:GND #PWR018
 U 1 1 5CCAA654
-P 6000 2050
-F 0 "#PWR018" H 6000 1800 50  0001 C CNN
-F 1 "GND" H 6005 1877 50  0000 C CNN
-F 2 "" H 6000 2050 50  0001 C CNN
-F 3 "" H 6000 2050 50  0001 C CNN
-	1    6000 2050
+P 6000 2150
+F 0 "#PWR018" H 6000 1900 50  0001 C CNN
+F 1 "GND" H 6005 1977 50  0000 C CNN
+F 2 "" H 6000 2150 50  0001 C CNN
+F 3 "" H 6000 2150 50  0001 C CNN
+	1    6000 2150
 	1    0    0    -1
 $EndComp
@@
 Wire Wire Line
 	6200 1750 5600 1750
+Text Label 5700 1750 0    50   ~ 0
+SYS_SWDIO
 Text Label 5700 1650 0    50   ~ 0
-SYS_SWDIO
-Text Label 5700 1750 0    50   ~ 0
 SYS_SWCLK
 NoConn ~ 5900 3650
@@
 	5900 3550 6500 3550
 $Comp
-L Connector:TestPoint TP2
+L Connector:TestPoint TP1
 U 1 1 5CAF561B
 P 6500 3550
-F 0 "TP2" V 6454 3738 50  0000 L CNN
-F 1 "OW-SYNC" V 6545 3738 50  0000 L CNN
+F 0 "TP1" V 6454 3738 50  0000 L CNN
+F 1 "SYNC" V 6545 3738 50  0000 L CNN
 F 2 "TestPoint:TestPoint_Pad_D1.5mm" H 6700 3550 50  0001 C CNN
 F 3 "~" H 6700 3550 50  0001 C CNN
@@
 OW-SYNC
 Wire Wire Line
-	2200 5650 2700 5650
-Wire Wire Line
-	2600 5550 2600 5850
-Connection ~ 2600 5550
-Wire Wire Line
-	2600 5550 3300 5550
-Wire Wire Line
-	2700 5850 2700 5650
-Connection ~ 2700 5650
-Wire Wire Line
-	2700 5650 3300 5650
-Wire Wire Line
-	2800 5350 2800 5850
-Connection ~ 2800 5350
-Wire Wire Line
 	9550 3100 9750 3100
 Wire Wire Line
@@
 	9750 3100 10250 3100
 $Comp
-L Device:LED D3
+L Device:LED D2
 U 1 1 5CD005A0
 P 5750 5900
-F 0 "D3" V 5789 5783 50  0000 R CNN
+F 0 "D2" V 5789 5783 50  0000 R CNN
 F 1 "LED2" V 5698 5783 50  0000 R CNN
 F 2 "LED_SMD:LED_0805_2012Metric" H 5750 5900 50  0001 C CNN
@@
 	0    -1   -1   0
 $EndComp
+Wire Wire Line
+	2700 5650 2700 5850
+Wire Wire Line
+	2800 5850 2800 5550
+Connection ~ 2800 5550
+Wire Wire Line
+	2800 5550 3300 5550
+Wire Wire Line
+	2200 5550 2800 5550
+Connection ~ 2700 5650
+Wire Wire Line
+	2700 5650 3300 5650
+Wire Wire Line
+	2200 5650 2700 5650
+Wire Wire Line
+	2600 5850 2600 5350
+Connection ~ 2600 5350
+Wire Wire Line
+	6200 1850 5600 1850
+Text Label 5700 1850 0    50   ~ 0
+NRST
+Text Label 4400 3150 0    50   ~ 0
+NRST
 $EndSCHEMATC

Commit message: New USB stick PCB design
Parts:
- removed D4: SP0503BAHT, Package_TO_SOT_SMD:SOT-143, symbol Power_Protection:SP0503BAHT
- removed J1: Pull-Up, Connector_PinHeader_2.54mm:PinHeader_1x02_P2.54mm_Vertical, symbol Connector_Generic:Conn_01x02
- removed J3: USB_B_Micro, Connector_USB:USB_Micro-B_Molex-105017-0001, symbol Connector:USB_B_Micro
- added FID1, FID2: Fiducial, Fiducial:Fiducial_0.5mm_Mask1.5mm, symbol Mechanical:Fiducial
- added J2: USB_A, Connector_USB:USB_A_CNCTech_1001-011-01101_Horizontal, symbol Connector:USB_A
- added JP1: PUP, Jumper:SolderJumper-2_P1.3mm_Open_RoundedPad1.0x1.5mm, symbol Jumper:SolderJumper_2_Open
- added U1: USBLC6-2SC6, Package_TO_SOT_SMD:SOT-23-6, symbol Power_Protection:USBLC6-2SC6
- C3: renamed from C2; footprint Capacitor_SMD:C_0805_2012Metric -> Capacitor_SMD:C_0603_1608Metric; Part Number CL21B225KAFNNNE -> CL10A225KO8NNNC
- C4: renamed from C1; footprint Capacitor_SMD:C_0805_2012Metric -> Capacitor_SMD:C_0603_1608Metric; Part Number CL21B105KBFNNNE -> CL10A105KO8NNNC
- D1: footprint LED_SMD:LED_0805_2012Metric -> LED_SMD:LED_0603_1608Metric; Part Number LTST-C170KGKT -> LTST-C190KGKT
- D2: footprint LED_SMD:LED_0805_2012Metric -> LED_SMD:LED_0603_1608Metric; Part Number LTST-C170KRKT -> LTST-C191KRKT
- F1: footprint Fuse:Fuse_1206_3216Metric -> Fuse:Fuse_0805_2012Metric; Part Number MF-NSMF012-2 -> MF-PSMF010X-2
- J1: renamed from J2; footprint Connector_JST:JST_XH_B02B-XH-A_1x02_P2.50mm_Vertical -> Connector_PinHeader_2.54mm:PinHeader_1x02_P2.54mm_Vertical; Brand KLS ELECTRONIC -> (none); Part Number L-KLS1-2.50-02-S -> (none)
- JP2: renamed from SW1; value BOOT -> DFU; footprint Button_Switch_SMD:SW_SPST_CK_RS282G05A3 -> Jumper:SolderJumper-2_P1.3mm_Open_RoundedPad1.0x1.5mm; symbol Switch:SW_Push -> Jumper:SolderJumper_2_Open; Brand KLS ELECTRONIC -> (none); Part Number L-KLS7-TS3611-2.5-180-T -> (none)
- R3: renamed from R1; Part Number 0603SAJ0222T5E -> 0805S8J0222T5E
- TP1, TP2: footprint TestPoint:TestPoint_Pad_D1.5mm -> TestPoint:TestPoint_Pad_D1.0mm
- renumbered C3 to C1, C4 to C2, J4 to J3, R2 to R1, R3 to R2, R7 to R6, R6 to R7, U1 to U3
Connections:
- net labels added: USB1_DN, USB1_DP, USB_DN, USB_DP
- net labels removed: OW-5V, USB_N, USB_P
- wire segments 99 -> 96
- no-connect marks 7 -> 6
Other:
- moved on the sheet: C1, C2, C3, C4, D1, D2, D3, F1, J1, J3, Q1, R1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
